File: bb1.kicad_pcb (KiCad board)
At the start: 2 copper layers, 331.5 x 112.1 mm, 154 parts, among them J1 USB_A, J2 ER-TFT035, J3 expansion, J4 ER-TFT032, J5 amp, J6 TOUCH_T, Q1 Q_Photo_NPN, SW1 SW_SPST, SW10 SW_SPST, SW11 SW_SPST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

Commit message: Last changes, finally committed.
Parts:
- added ?: , , F.Cu at (-110.0, -67.2)
Connections:
- J5 pad 4: /DAC0 -> (no net)
- J5 pad 5: (no net) -> /DAC0
Routing:
- net /DAC0: track 16.2 -> 18.7 mm
Other:
- board text added: "TODO: Add part numbers of switches to front silkscreen, add labels to reset/programming switches"
