File: bb1.sch (KiCad schematic (older format))
At the start: 154 parts, among them J1 USB_A, J2 ER-TFT035, J3 expansion, J4 ER-TFT032, J5 amp, J6 TOUCH_T, Q1 Q_Photo_NPN, SW1 SW_SPST, SW10 SW_SPST, SW11 SW_SPST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

Commit message: Last changes, finally committed.
Other:
- note added: "ANODES/POSITIVE"
- note added: "CATHODES/NEGATIVE"
- moved on the sheet: J2, J3, J4, J5
